Commit message: .

File: system_model/payload/box/box.urdf (robot description, URDF)
Before this commit: robot payload, 4 links, 3 joints
Links:
- link payload: mass 1.0 -> 0.4; geometry collision box size=0.2 0.2 0.05; visual box size=0.020999999999999998 0.020999999999999998 0.01
Joints:
- joint attach_0_joint: origin xyz=0.135 0.0 0.05 rpy=0 0 0 -> xyz=0.09000000000000001 0.0 0.025 rpy=0 0 0
- joint attach_1_joint: origin xyz=-0.06749999999999998 0.11691342951089924 0.05 rpy=0 0 0 -> xyz=-0.044999999999999984 0.07794228634059949 0.025 rpy=0 0 0
- joint attach_2_joint: origin xyz=-0.06750000000000006 -0.11691342951089918 0.05 rpy=0 0 0 -> xyz=-0.04500000000000005 -0.07794228634059946 0.025 rpy=0 0 0
